Commit message: adjust param

File: kortex_description/arms/gen3/6dof/urdf/gen3_macro.xacro (robot description, xacro)
@@ -4,5 +4,5 @@
   <xacro:property name="last_arm_link" value="end_effector_link"/>
   <xacro:macro name="load_arm" params="parent:='' dof vision prefix *origin">
-    <link name="${prefix}base_link">
+    <link name="arm_base_link">
       <inertial>
         <origin xyz="-0.000648 -0.000166 0.084487" rpy="0 0 0" />
@@ -50,5 +50,5 @@
     <joint name="${prefix}joint_1" type="continuous">
       <origin xyz="0 0 0.15643" rpy="-3.1416 0.0 0.0" />
-      <parent link="${prefix}base_link" />
+      <parent link="arm_base_link" />
       <child link="${prefix}shoulder_link" />
       <axis xyz="0 0 1" />
